Commit message: vehicle driving in gazebo (params still not working)

File: description/tank.urdf.xacro (robot description, xacro)
@@ -49,6 +49,6 @@
             </geometry>
         </collision>
-        <xacro:inertial_box mass="0.5" x="${chassis_length}" y="${chassis_width}" z="${chassis_height}">
-            <origin xyz="${chassis_length/2} 0 ${chassis_height/2}" rpy="0 0 0"/>
+        <xacro:inertial_box mass="2.0" x="${chassis_length}" y="${chassis_width}" z="${chassis_height}">
+            <origin xyz="$0 0 ${chassis_height}" rpy="0 0 0"/>
         </xacro:inertial_box>
     </link>
